Commit message: agg

File: src/model_arm/modello/model_arm_giusto.urdf (robot description, URDF)
Before this commit: robot arm, 9 links, 8 joints
Joints:
- joint plan_move: limit lower=0 upper=-0.55 effort=1000.0 velocity=0.5 -> lower=-0.55 upper=-0.05 effort=1000.0 velocity=0.5

Commit message: agg

File: src/model_arm/modello/model_arm_giusto.urdf (robot description, URDF)
Before this commit: robot arm, 9 links, 8 joints
Links:
- link base_link: geometry collision box size=0.088 0.090 0.029; visual box size=0.088 0.090 0.029
- link base_up: geometry collision box size=0.059 0.026 0.054; visual box size=0.059 0.026 0.054
- link connection_servo12: geometry collision box size=0.13 0.06 0.026; visual box size=0.13 0.06 0.026
- link connection_servo23: geometry collision box size=1.30 0.60 0.55; visual box size=0.130 0.060 0.055
- link gripper_b: geometry collision box size=0.050 0.072 0.052; visual box size=0.050 0.072 0.052
- link left_g: geometry collision box size=0.037 0.019 0.020; visual box size=0.037 0.019 0.020
- link right_g: geometry collision box size=0.037 0.019 0.020; visual box size=0.037 0.019 0.020
- link servo_arm_rotation: geometry collision box size=0.085 0.060 0.025; visual box size=0.085 0.060 0.025
- link servo_rotz: geometry collision box size=0.058 0.060 0.025; visual box size=0.058 0.060 0.025
Joints:
- joint baseup_link: origin xyz=0.205 0.03 0.405 -> xyz=0.0155 0 0.0415
- joint con_up_1: origin xyz=-0.05 0 0.045 -> xyz=-0.009 -0.013 0
- joint con_up_2: origin xyz= -1.04 0 0 -> xyz=-0.104 0 0
- joint con_up_3: origin xyz=-1.43 0 0 -> xyz=-0.094 0 0
- joint fix_left: origin xyz=-0.375 0.225 0 -> xyz=-0.068 -0.038 0
- joint plan_move: limit lower=-0.55 upper=-0.05 effort=1000.0 velocity=0.5 -> lower=0 upper=0.053 effort=1000.0 velocity=0.5; origin xyz=0 -0.15 0 -> xyz=0 0.019 0
- joint rotation_grip: origin xyz=-0.74 0 0 -> xyz=-0.072 0.013 0
- joint servo_link2: origin xyz=0.11 -0.01 0.38 -> xyz=0.0095 0 0.0395
