Commit message: fix double

File: src/braccio_simulation/model/urdf/inc/create_link.xacro (robot description, xacro)
@@ -1,5 +1,29 @@
 <?xml version="1.0"?>
 <robot xmlns:xacro="http://wiki.ros.org/xacro">
-  <xacro:macro name="create_link" params="
+  <xacro:macro name="create_link_from_box" params="
+        link_name
+        xyz_offset
+        rpy_offset
+        dim_box">
+    <link name="${link_name}">
+      <visual>
+        <origin xyz="${xyz_offset}" rpy="${rpy_offset}"/>
+        <geometry>
+          <box size="${dim_box}"/>
+        </geometry>
+      </visual>
+      <collision>
+        <origin xyz="${xyz_offset}" rpy="${rpy_offset}"/>
+        <geometry>
+          <box size="${dim_box}"/>
+        </geometry>
+      </collision>
+      <inertial>
+        <mass value="1"/>
+        <inertia ixx="1.0" ixy="0.0" ixz="0.0" iyy="1.0" iyz="0.0" izz="1.0"/>
+      </inertial>
+    </link>
+  </xacro:macro>
+  <xacro:macro name="create_link_from_mesh" params="
         link_name
         xyz_offset
@@ -11,5 +35,5 @@
         <origin xyz="${xyz_offset}" rpy="${rpy_offset}"/>
         <geometry>
-          <mesh filename="package://${mesh_package}/meshes/visual/${mesh_name}.dae"/>
+          <mesh filename="package://${mesh_package}/${mesh_name}.dae" scale="0.001 0.001 0.001"/>
         </geometry>
       </visual>
@@ -17,5 +41,5 @@
         <origin xyz="${xyz_offset}" rpy="${rpy_offset}"/>
         <geometry>
-          <mesh filename="package://${mesh_package}/meshes/collision/${mesh_name}.stl"/>
+          <mesh filename="package://${mesh_package}/${mesh_name}.stl" scale="0.001 0.001 0.001"/>
         </geometry>
       </collision>
