Commit message: add new xacro macro for link

File: src/braccio_simulation/model/urdf/braccio.urdf.xacro (robot description, xacro)
@@ -3,59 +3,82 @@
   <xacro:macro name="r6bot_description">
   <!-- Load the YAML file -->
-  <!--
-  <xacro:property name="yaml_file" value="$(find ros2_sim_description)/config/rrr.yaml"/>
-  <xacro:property name="robot_measures" value="${xacro.load_yaml(yaml_file)}"/>
-  <xacro:property name="box_base_length" value="${robot_measures['box_base']['length']}"/>
-  -->
+  <!-- <xacro:property name="yaml_file" value="$(find braccio_simulation)/urdf/config/braccio_param.yaml"/>
+  <xacro:property name="robot_descr" value="${xacro.load_yaml(yaml_file)}"/> -->
   <!-- helper macro -->
-  <xacro:include filename="$(find ros2_control_demo_description)/r6bot/urdf/inc/create_link.xacro"/>
-  <xacro:create_link
+  <xacro:include filename="$(find braccio_simulation)/model/urdf/inc/create_link.xacro"/>
+  <xacro:create_link_from_box
       link_name="base_link"
+      xyz_offset="0 0 0.0145"
+      rpy_offset="0 0 0"
+      dim_box="0.088 0.090 0.029"
+  />
+  <xacro:create_link_from_box
+      link_name="base_up"
       xyz_offset="0 0 0"
       rpy_offset="0 0 0"
-      mesh_package="ros2_control_demo_description/r6bot"
-      mesh_name="link_0"
+      dim_box="0.059 0.026 0.050"
   />
-  <xacro:create_link
-      link_name="link_1"
-      xyz_offset="0 0 -0.182"
+  <xacro:create_link_from_box
+      link_name="arm_rot"
+      xyz_offset="0.002 0.012 0.013"
       rpy_offset="0 0 0"
-      mesh_package="ros2_control_demo_description/r6bot"
-      mesh_name="link_1"
+      dim_box="0.058 0.050 0.026"
   />
-  <xacro:create_link
-      link_name="link_2"
-      xyz_offset="0 0 -0.168"
+  <xacro:create_link_from_mesh
+      link_name="arm_1_up_down_p1"
+      xyz_offset="0 0 0"
+      rpy_offset="0 0 -${pi2}"
+      mesh_package="model/3Dparts"
+      mesh_name="ModelARM-Body.stl"
+  />
+  <xacro:create_link_from_mesh
+      link_name="arm_1_up_down_p2"
+      xyz_offset="0 0 0"
+      rpy_offset="${pi} 0 -${pi2}"
+      mesh_package="model/3Dparts"
+      mesh_name="ModelARM-Body.stl"
+  />
+  <xacro:create_link_from_box
+      link_name="arm_2_up_down"
+      xyz_offset="0.045 -0.001 0"
       rpy_offset="0 0 0"
-      mesh_package="ros2_control_demo_description/r6bot"
-      mesh_name="link_2"
+      dim_box="0.13 0.050 0.028"
   />
-  <xacro:create_link
-      link_name="link_3"
-      xyz_offset="0 0 -0.144"
+  <xacro:create_link_from_mesh
+      link_name="arm_3_up_down"
+      xyz_offset="0 0 0"
+      rpy_offset="0 0 -${pi2}"
+      mesh_package="model/3Dparts"
+      mesh_name="ModelARM-Body.stl"
+  />
+  <xacro:create_link_from_box
+      link_name="box_servo_rot"
+      xyz_offset="0 0 0"
       rpy_offset="0 0 0"
-      mesh_package="ros2_control_demo_description/r6bot"
-      mesh_name="link_3"
+      dim_box="0.042 0.042 0.021"
   />
-  <xacro:create_link
-      link_name="link_4"
-      xyz_offset="0 0 0.077"
+  <xacro:create_link_from_box
+      link_name="rot_grasp"
+      xyz_offset="0.0265 0 0"
       rpy_offset="0 0 0"
-      mesh_package="ros2_control_demo_description/r6bot"
-      mesh_name="link_4"
+      dim_box="0.053 0.055 0.019"
   />
-  <xacro:create_link
-      link_name="link_5"
-      xyz_offset="0 0 0.113"
+  <xacro:create_link_from_box
+      link_name="grasp_box"
+      xyz_offset="0.03 0.025 0.0165"
       rpy_offset="0 0 0"
-      mesh_package="ros2_control_demo_description/r6bot"
-      mesh_name="link_5"
+      dim_box="0.020 0.050 0.033"
   />
-  <xacro:create_link
-      link_name="link_6"
-      xyz_offset="0 0 0.086"
+  <xacro:create_link_from_box
+      link_name="grasp_l"
+      xyz_offset="0.029 0.005 0"
       rpy_offset="0 0 0"
-      mesh_package="ros2_control_demo_description/r6bot"
-      mesh_name="link_6"
+      dim_box="0.058 0.010 0.020"
+  />
+  <xacro:create_link_from_box
+      link_name="grasp_r"
+      xyz_offset="0.029 -0.005 0"
+      rpy_offset="0 0 0"
+      dim_box="0.058 0.010 0.020"
   />
   <link name="ft_frame"/>

File: src/braccio_simulation/model/urdf/inc/create_link.xacro (robot description, xacro)
@@ -35,5 +35,5 @@
         <origin xyz="${xyz_offset}" rpy="${rpy_offset}"/>
         <geometry>
-          <mesh filename="package://${mesh_package}/${mesh_name}.dae" scale="0.001 0.001 0.001"/>
+          <mesh filename="package://${mesh_package}/${mesh_name}.stl" scale="0.001 0.001 0.001"/>
         </geometry>
       </visual>

File: src/braccio_simulation/model/urdf/model_braccio.urdf (robot description, URDF)
Before this commit: robot braccio, 12 links, 11 joints
Joints:
- joint supServoRot: axis 0 1 0 -> (none); limit lower=-${pi2} upper=${pi2} effort=1000.0 velocity=0.5 -> (none)

Commit message: update urdf with xacro

File: src/braccio_simulation/model/urdf/braccio.urdf.xacro (robot description, xacro)
@@ -1,147 +1,8 @@
 <?xml version="1.0"?>
-<robot xmlns:xacro="http://www.ros.org/wiki/xacro">
-  <xacro:macro name="r6bot_description">
-  <!-- Load the YAML file -->
-  <!-- <xacro:property name="yaml_file" value="$(find braccio_simulation)/urdf/config/braccio_param.yaml"/>
-  <xacro:property name="robot_descr" value="${xacro.load_yaml(yaml_file)}"/> -->
-  <!-- helper macro -->
-  <xacro:include filename="$(find braccio_simulation)/model/urdf/inc/create_link.xacro"/>
-  <xacro:create_link_from_box
-      link_name="base_link"
-      xyz_offset="0 0 0.0145"
-      rpy_offset="0 0 0"
-      dim_box="0.088 0.090 0.029"
-  />
-  <xacro:create_link_from_box
-      link_name="base_up"
-      xyz_offset="0 0 0"
-      rpy_offset="0 0 0"
-      dim_box="0.059 0.026 0.050"
-  />
-  <xacro:create_link_from_box
-      link_name="arm_rot"
-      xyz_offset="0.002 0.012 0.013"
-      rpy_offset="0 0 0"
-      dim_box="0.058 0.050 0.026"
-  />
-  <xacro:create_link_from_mesh
-      link_name="arm_1_up_down_p1"
-      xyz_offset="0 0 0"
-      rpy_offset="0 0 -${pi2}"
-      mesh_package="model/3Dparts"
-      mesh_name="ModelARM-Body.stl"
-  />
-  <xacro:create_link_from_mesh
-      link_name="arm_1_up_down_p2"
-      xyz_offset="0 0 0"
-      rpy_offset="${pi} 0 -${pi2}"
-      mesh_package="model/3Dparts"
-      mesh_name="ModelARM-Body.stl"
-  />
-  <xacro:create_link_from_box
-      link_name="arm_2_up_down"
-      xyz_offset="0.045 -0.001 0"
-      rpy_offset="0 0 0"
-      dim_box="0.13 0.050 0.028"
-  />
-  <xacro:create_link_from_mesh
-      link_name="arm_3_up_down"
-      xyz_offset="0 0 0"
-      rpy_offset="0 0 -${pi2}"
-      mesh_package="model/3Dparts"
-      mesh_name="ModelARM-Body.stl"
-  />
-  <xacro:create_link_from_box
-      link_name="box_servo_rot"
-      xyz_offset="0 0 0"
-      rpy_offset="0 0 0"
-      dim_box="0.042 0.042 0.021"
-  />
-  <xacro:create_link_from_box
-      link_name="rot_grasp"
-      xyz_offset="0.0265 0 0"
-      rpy_offset="0 0 0"
-      dim_box="0.053 0.055 0.019"
-  />
-  <xacro:create_link_from_box
-      link_name="grasp_box"
-      xyz_offset="0.03 0.025 0.0165"
-      rpy_offset="0 0 0"
-      dim_box="0.020 0.050 0.033"
-  />
-  <xacro:create_link_from_box
-      link_name="grasp_l"
-      xyz_offset="0.029 0.005 0"
-      rpy_offset="0 0 0"
-      dim_box="0.058 0.010 0.020"
-  />
-  <xacro:create_link_from_box
-      link_name="grasp_r"
-      xyz_offset="0.029 -0.005 0"
-      rpy_offset="0 0 0"
-      dim_box="0.058 0.010 0.020"
-  />
-  <link name="ft_frame"/>
-  <link name="tool0"/>
-  <!-- base_joint fixes base_link to the environment -->
-  <joint name="base_joint" type="fixed">
-    <parent link="world"/>
-    <child link="base_link"/>
-    <origin xyz="0 0 0" rpy="0 0 0"/>
-    <axis xyz="0 0 1"/>
-  </joint>
-  <!-- joints - main serial chain -->
-  <joint name="joint_1" type="revolute">
-    <parent link="base_link"/>
-    <child link="link_1"/>
-    <origin xyz="0 0 0.244" rpy="0 0 0"/>
-    <axis xyz="0 0 1"/>
-    <limit effort="1000.0" lower="${-pi}" upper="${pi}" velocity="2.5"/>
-  </joint>
-  <joint name="joint_2" type="revolute">
-    <parent link="link_1"/>
-    <child link="link_2"/>
-    <origin xyz="-0.27 0 0.0" rpy="${-pi/2} -${pi/2} ${pi/2}"/>
-    <axis xyz="0 0 1"/>
-    <limit effort="1000.0" lower="${-pi}" upper="${pi}" velocity="2.5"/>
-  </joint>
-  <joint name="joint_3" type="revolute">
-    <parent link="link_2"/>
-    <child link="link_3"/>
-    <origin xyz="0.686 0 -0.27" rpy="0 ${pi} ${pi+pi/2}"/>
-    <axis xyz="0 0 1"/>
-    <limit effort="1000.0" lower="${-pi}" upper="${pi}" velocity="2.5"/>
-  </joint>
-  <joint name="joint_4" type="revolute">
-    <parent link="link_3"/>
-    <child link="link_4"/>
-    <origin xyz="0.519 0 0" rpy="0 ${pi} ${pi}"/>
-    <axis xyz="0 0 1"/>
-    <limit effort="1000.0" lower="${-pi}" upper="${pi}" velocity="2.5"/>
-  </joint>
-  <joint name="joint_5" type="revolute">
-    <parent link="link_4"/>
-    <child link="link_5"/>
-    <origin xyz="0.0 0 0.188" rpy="${pi/2} ${pi} ${pi/2}"/>
-    <axis xyz="0 0 1"/>
-    <limit effort="1000.0" lower="${-pi}" upper="${pi}" velocity="2.5"/>
-  </joint>
-  <joint name="joint_6" type="revolute">
-    <parent link="link_5"/>
-    <child link="link_6"/>
-    <origin xyz="0.0 0 0.246" rpy="0 ${-pi/2} 0"/>
-    <axis xyz="0 0 1"/>
-    <limit effort="1000.0" lower="${-pi}" upper="${pi}" velocity="2.5"/>
-  </joint>
-  <joint name="joint-ft_frame" type="fixed">
-    <parent link="link_6"/>
-    <child link="ft_frame"/>
-    <origin xyz="0 0 0.086" rpy="0 0 0"/>
-  </joint>
-  <joint name="joint-tool" type="fixed">
-    <parent link="ft_frame"/>
-    <child link="tool0"/>
-    <origin xyz="0 0 0.185" rpy="0 0 0"/>
-  </joint>
-</xacro:macro>
+<robot xmlns:xacro="http://wiki.ros.org/xacro" name="braccio">
+  <!-- Import r6bot macro -->
+  <xacro:include filename="$(find braccio_simulation)/model/urdf/braccio_description.urdf.xacro"/>
+  <!-- create link fixed to the "world" -->
+  <link name="world"/>
+  <xacro:braccio_description/>
 </robot>

File: src/braccio_simulation/model/urdf/inc/create_link.xacro (robot description, xacro)
@@ -35,5 +35,5 @@
         <origin xyz="${xyz_offset}" rpy="${rpy_offset}"/>
         <geometry>
-          <mesh filename="package://${mesh_package}/${mesh_name}.stl" scale="0.001 0.001 0.001"/>
+          <mesh filename="file://${mesh_package}/${mesh_name}" scale="0.001 0.001 0.001"/>
         </geometry>
       </visual>
@@ -41,5 +41,5 @@
         <origin xyz="${xyz_offset}" rpy="${rpy_offset}"/>
         <geometry>
-          <mesh filename="package://${mesh_package}/${mesh_name}.stl" scale="0.001 0.001 0.001"/>
+          <mesh filename="file://${mesh_package}/${mesh_name}" scale="0.001 0.001 0.001"/>
         </geometry>
       </collision>
