Commit message: more doc

File: src/braccio_control/description/ros2_control/braccio.ros2_control.xacro (robot description, xacro)
@@ -1,10 +1,10 @@
 <?xml version="1.0"?>
 <robot xmlns:xacro="http://www.ros.org/wiki/xacro">
-  <xacro:macro name="r6bot_ros2_control" params="name">
+  <xacro:macro name="braccio_ros2_control" params="name">
     <ros2_control name="${name}" type="system">
       <hardware>
-        <plugin>ros2_control_demo_example_7/RobotSystem</plugin>
+        <plugin>ros2_control_braccio/RobotSystem</plugin>
       </hardware>
-      <joint name="joint_1">
+      <joint name="arm_rot">
         <command_interface name="position">
           <param name="min">${-2*pi}</param>
@@ -20,5 +20,5 @@
         <state_interface name="velocity"/>
       </joint>
-      <joint name="joint_2">
+      <joint name="arm_1_up_down">
         <command_interface name="position">
           <param name="min">${-2*pi}</param>
@@ -34,5 +34,5 @@
         <state_interface name="velocity"/>
       </joint>
-      <joint name="joint_3">
+      <joint name="arm_2_up_down">
         <command_interface name="position">
           <param name="min">${-pi}</param>
@@ -48,5 +48,5 @@
         <state_interface name="velocity"/>
       </joint>
-      <joint name="joint_4">
+      <joint name="arm_3_up_down">
         <command_interface name="position">
           <param name="min">${-2*pi}</param>
@@ -62,5 +62,5 @@
         <state_interface name="velocity"/>
       </joint>
-      <joint name="joint_5">
+      <joint name="rot_grasp">
         <command_interface name="position">
           <param name="min">${-2*pi}</param>
@@ -76,5 +76,5 @@
         <state_interface name="velocity"/>
       </joint>
-      <joint name="joint_6">
+      <joint name="grasp">
         <command_interface name="position">
           <param name="min">${-2*pi}</param>
@@ -90,12 +90,4 @@
         <state_interface name="velocity"/>
       </joint>
-      <sensor name="tcp_fts_sensor">
-        <state_interface name="force.x"/>
-        <state_interface name="force.y"/>
-        <state_interface name="force.z"/>
-        <state_interface name="torque.x"/>
-        <state_interface name="torque.y"/>
-        <state_interface name="torque.z"/>
-      </sensor>
     </ros2_control>
   </xacro:macro>

File: src/braccio_control/description/urdf/braccio.urdf.xacro (robot description, xacro)
@@ -2,5 +2,5 @@
 <robot xmlns:xacro="http://wiki.ros.org/xacro" name="braccio">
   <!-- Import r6bot macro -->
-  <xacro:include filename="$(find braccio_simulation)/urdf/braccio.urdf"/>
+  <xacro:include filename="$(find braccio_simulation)/model/urdf/braccio.urdf.xacro"/>
   <!-- create link fixed to the "world" -->
   <link name="world"/>

Commit message: add zenoh

File: src/braccio_control/description/ros2_control/braccio.ros2_control.xacro (robot description, xacro)
@@ -2,4 +2,5 @@
 <robot xmlns:xacro="http://www.ros.org/wiki/xacro">
   <xacro:macro name="braccio_ros2_control" params="name">
+    <xacro:property name="pi2" value="1.570796327" />
     <ros2_control name="${name}" type="system">
       <hardware>
@@ -8,6 +9,6 @@
       <joint name="arm_rot">
         <command_interface name="position">
-          <param name="min">${-2*pi}</param>
-          <param name="max">${2*pi}</param>
+          <param name="min">-${pi2}</param>
+          <param name="max">${pi2}</param>
         </command_interface>
         <state_interface name="position">
@@ -17,6 +18,6 @@
       <joint name="arm_1_up_down">
         <command_interface name="position">
-          <param name="min">${-2*pi}</param>
-          <param name="max">${2*pi}</param>
+          <param name="min">-${pi2}</param>
+          <param name="max">${pi2}</param>
         </command_interface>
         <state_interface name="position">
@@ -26,6 +27,6 @@
       <joint name="arm_2_up_down">
         <command_interface name="position">
-          <param name="min">${-pi}</param>
-          <param name="max">${pi}</param>
+          <param name="min">-${pi2}</param>
+          <param name="max">${pi2}</param>
         </command_interface>
         <state_interface name="position">
@@ -35,6 +36,6 @@
       <joint name="arm_3_up_down">
         <command_interface name="position">
-          <param name="min">${-2*pi}</param>
-          <param name="max">${2*pi}</param>
+          <param name="min">-${pi2}</param>
+          <param name="max">${pi2}</param>
         </command_interface>
         <state_interface name="position">
@@ -44,6 +45,6 @@
       <joint name="rot_grasp">
         <command_interface name="position">
-          <param name="min">${-2*pi}</param>
-          <param name="max">${2*pi}</param>
+          <param name="min">-${pi2}</param>
+          <param name="max">${pi2}</param>
         </command_interface>
         <state_interface name="position">
@@ -51,13 +52,23 @@
         </state_interface>
       </joint>
-      <joint name="grasp">
+    <joint name="grasp">
         <command_interface name="position">
-          <param name="min">${-2*pi}</param>
-          <param name="max">${2*pi}</param>
+          <param name="min">0</param>
+          <param name="max">0.03</param>
+        </command_interface>
+      <state_interface name="position"/>
+    </joint>
+    <joint name="grasp_mirror">
+      <state_interface name="position"/>
+    </joint>
+      <!-- <joint name="grasp">
+        <command_interface name="position">
+          <param name="min">-${pi2}</param>
+          <param name="max">${pi2}</param>
         </command_interface>
         <state_interface name="position">
           <param name="initial_value">0.0</param>
         </state_interface>
-      </joint>
+      </joint> -->
     </ros2_control>
   </xacro:macro>

File: src/braccio_simulation/model/urdf/braccio_description.urdf.xacro (robot description, xacro)
@@ -143,5 +143,5 @@
       <origin xyz="0 0 0"/>
     </joint>
-    <joint name="grasp" type="prismatic">
+    <joint name="grasp_ctrl" type="prismatic">
       <axis xyz="0 1 0"/>
       <limit
@@ -154,5 +154,5 @@
       <origin xyz="0.052 0 0"/>
     </joint>
-    <joint name="plan_move" type="prismatic">
+    <joint name="grasp_mirror" type="prismatic">
       <axis xyz="0 -1 0"/>
       <limit
@@ -165,5 +165,5 @@
       <origin xyz="0.052 0 0"/>
       <mimic
-        joint="grasp"
+        joint="grasp_ctrl"
         multiplier="1"
         offset="0" />

Commit message: fix controller

File: src/braccio_control/description/ros2_control/braccio.ros2_control.xacro (robot description, xacro)
@@ -5,5 +5,5 @@
     <ros2_control name="${name}" type="system">
       <hardware>
-        <plugin>ros2_control_braccio/RobotSystem</plugin>
+        <plugin>braccio_control/RobotSystem</plugin>
       </hardware>
       <joint name="arm_rot">
@@ -52,5 +52,5 @@
         </state_interface>
       </joint>
-    <joint name="grasp">
+    <joint name="grasp_ctrl">
         <command_interface name="position">
           <param name="min">0</param>
@@ -59,16 +59,7 @@
       <state_interface name="position"/>
     </joint>
-    <joint name="grasp_mirror">
+    <!-- <joint name="grasp_mirror">
       <state_interface name="position"/>
-    </joint>
-      <!-- <joint name="grasp">
-        <command_interface name="position">
-          <param name="min">-${pi2}</param>
-          <param name="max">${pi2}</param>
-        </command_interface>
-        <state_interface name="position">
-          <param name="initial_value">0.0</param>
-        </state_interface>
-      </joint> -->
+    </joint> -->
     </ros2_control>
   </xacro:macro>

File: src/braccio_simulation/model/urdf/braccio_description.urdf.xacro (robot description, xacro)
@@ -169,4 +169,10 @@
         offset="0" />
     </joint>
+  <link name="tool0"/>
+  <joint name="joint-tool" type="fixed">
+    <parent link="rot_grasp"/>
+    <child link="tool0"/>
+    <origin xyz="0.07 0 0" rpy="0 0 0"/>
+  </joint>
   </xacro:macro>
 </robot>
