Commit message: impr

File: src/braccio_moveit/config/braccio.ros2_control.xacro (robot description, xacro)
@@ -13,4 +13,5 @@
                   <param name="initial_value">${initial_positions['arm_rot']}</param>
                 </state_interface>
+                <state_interface name="velocity"/>
             </joint>
             <joint name="arm_1_up_down">
@@ -19,4 +20,5 @@
                   <param name="initial_value">${initial_positions['arm_1_up_down']}</param>
                 </state_interface>
+                <state_interface name="velocity"/>
             </joint>
             <joint name="arm_2_up_down">
@@ -25,4 +27,5 @@
                   <param name="initial_value">${initial_positions['arm_2_up_down']}</param>
                 </state_interface>
+                <state_interface name="velocity"/>
             </joint>
             <joint name="arm_3_up_down">
@@ -31,4 +34,5 @@
                   <param name="initial_value">${initial_positions['arm_3_up_down']}</param>
                 </state_interface>
+                <state_interface name="velocity"/>
             </joint>
             <joint name="rot_grasp">
@@ -37,4 +41,5 @@
                   <param name="initial_value">${initial_positions['rot_grasp']}</param>
                 </state_interface>
+                <state_interface name="velocity"/>
             </joint>
             <joint name="grasp_ctrl">
@@ -43,4 +48,5 @@
                   <param name="initial_value">${initial_positions['grasp_ctrl']}</param>
                 </state_interface>
+                <state_interface name="velocity"/>
             </joint>
         </ros2_control>

File: src/braccio_simulation/model/urdf/braccio_description.urdf.xacro (robot description, xacro)
@@ -95,5 +95,5 @@
     <joint name="arm_rot" type="revolute">
       <axis xyz="0 0 1"/>
-      <limit effort="1000.0" lower="-${pi2}" upper="${pi2}" velocity="0.5"/>
+      <limit effort="1000.0" lower="-${pi2}" upper="${pi2}" velocity="0.5" acceleration="1.0"/>
       <parent link="base_vert_servo_rot"/>
       <child link="base_servo_ud"/>
@@ -102,5 +102,5 @@
     <joint name="arm_1_up_down" type="revolute">
       <axis xyz="0 1 0"/>
-      <limit effort="1000.0" lower="-${pi2}" upper="${pi2}" velocity="0.5"/>
+      <limit effort="1000.0" lower="-${pi2}" upper="${pi2}" velocity="0.5" acceleration="1.0"/>
       <parent link="base_servo_ud"/>
       <child link="arm_1_up_down_p1"/>
@@ -114,5 +114,5 @@
     <joint name="arm_2_up_down" type="revolute">
       <axis xyz="0 1 0"/>
-      <limit effort="1000.0" lower="-${pi2}" upper="${pi2}" velocity="0.5"/>
+      <limit effort="1000.0" lower="-${pi2}" upper="${pi2}" velocity="0.5" acceleration="1.0"/>
       <parent link="arm_1_up_down_p2"/>
       <child link="arm_2_up_down"/>
@@ -121,5 +121,5 @@
     <joint name="arm_3_up_down" type="revolute">
       <axis xyz="0 1 0"/>
-      <limit effort="1000.0" lower="-${pi2}" upper="${pi2}" velocity="0.5"/>
+      <limit effort="1000.0" lower="-${pi2}" upper="${pi2}" velocity="0.5" acceleration="1.0"/>
       <parent link="arm_2_up_down"/>
       <child link="arm_3_up_down"/>
@@ -133,5 +133,5 @@
     <joint name="rot_grasp" type="revolute">
       <axis xyz="1 0 0"/>
-      <limit effort="1000.0" lower="-${pi2}" upper="${pi2}" velocity="0.5"/>
+      <limit effort="1000.0" lower="-${pi2}" upper="${pi2}" velocity="0.5" acceleration="1.0"/>
       <parent link="box_servo_rot"/>
       <child link="rot_grasp"/>
@@ -149,4 +149,5 @@
         upper="0.03"
         velocity="2.0"
+        acceleration="1.0"
         effort="1000" />
       <parent link="rot_grasp"/>
@@ -160,4 +161,5 @@
         upper="0.03"
         velocity="2.0"
+         acceleration="1.0"
         effort="1000" />
       <parent link="rot_grasp"/>
@@ -175,4 +177,11 @@
     <origin xyz="0.07 0 0" rpy="0 0 0"/>
   </joint>
+  <link name="tool01"/>
+  <joint name="joint-tool01" type="fixed">
+    <parent link="box_servo_rot"/>
+    <child link="tool01"/>
+    <!-- 0.03 0.025 0.0165 -->
+    <origin xyz="0.098 -0.011 0" rpy="0 0 0"/>
+  </joint>
   </xacro:macro>
 </robot>
